Commit message: changed lower and upper limit.

File: gym-foodhunting/urdf/r2d2.urdf (robot description, URDF)
Before this commit: robot physics, 16 links, 15 joints
Joints:
- joint head_swivel: limit lower=-3.14 upper=3.14 effort=1000.0 velocity=0.5 -> lower=-3.14159 upper=3.14159 effort=1000.0 velocity=0.5

Commit message: fixed gripper_extension's lower limit.

File: gym-foodhunting/urdf/r2d2.urdf (robot description, URDF)
Before this commit: robot physics, 16 links, 15 joints
Joints:
- joint gripper_extension: limit lower=-0.38 upper=0 effort=1000.0 velocity=0.5 -> lower=-0.17 upper=0 effort=1000.0 velocity=0.5
